Commit message: Updated robot description and added new launch/config files

File: description/robot.urdf.xacro (robot description, xacro)
@@ -1,5 +1,5 @@
 <?xml version="1.0"?>
 <robot xmlns:xacro="http://www.ros.org/wiki/xacro"  name="robot">
-   <xacro:arg name="use_ros2_control" default="true">
+   <xacro:arg name="use_ros2_control" default="true"/>
     <xacro:include filename="robot_core.xacro" />
     <xacro:if value="$(arg use_ros2_control)">

File: description/robot_core.xacro (robot description, xacro)
@@ -11,5 +11,5 @@
     <xacro:property name="wheel_offset_x" value="0.226"/>
     <xacro:property name="wheel_offset_y" value="0.166"/>
-    <xacro:property name="wheel_offset_z" value="0.01"/>
+    <xacro:property name="wheel_offset_z" value="${wheel_radius}"/>
     <xacro:property name="caster_wheel_radius" value="0.01"/>
     <xacro:property name="caster_wheel_mass" value="0.01"/>
@@ -74,5 +74,5 @@
         <child link="left_wheel"/>
         <origin xyz="0 ${wheel_offset_y} 0" rpy="-${pi/2} 0 0" />
-        <axis xyz="0 0 1"/>
+        <axis xyz="0 1 0"/>
     </joint>
     <link name="left_wheel">
@@ -83,9 +83,9 @@
             <material name="blue"/>
         </visual>
-        <collision>
-            <geometry>
-                <sphere radius="${wheel_radius}"/>
-            </geometry>
-        </collision>
+    <collision>
+        <geometry>
+            <cylinder radius="${wheel_radius}" length="${wheel_thickness}"/>
+        </geometry>
+    </collision>
         <xacro:inertial_cylinder mass="${wheel_mass}" length="${wheel_thickness}" radius="${wheel_radius}">
             <origin xyz="0 0 0" rpy="0 0 0"/>
@@ -100,5 +100,5 @@
         <child link="right_wheel"/>
         <origin xyz="0 ${-wheel_offset_y} 0" rpy="${pi/2} 0 0" />
-        <axis xyz="0 0 -1"/>
+        <axis xyz="0 -1 0"/>
     </joint>
     <link name="right_wheel">
@@ -109,9 +109,9 @@
             <material name="blue"/>
         </visual>
-        <collision>
-            <geometry>
-                <sphere radius="${wheel_radius}"/>
-            </geometry>
-        </collision>
+    <collision>
+        <geometry>
+            <cylinder radius="${wheel_radius}" length="${wheel_thickness}"/>
+        </geometry>
+    </collision>
         <xacro:inertial_cylinder mass="${wheel_mass}" length="${wheel_thickness}" radius="${wheel_radius}">
             <origin xyz="0 0 0" rpy="0 0 0"/>
@@ -145,6 +145,6 @@
     <gazebo reference="caster_wheel">
         <material>Gazebo/White</material>
-        <mu1 value="0.001"/>
-        <mu2 value="0.001"/>
+        <mu1 value="0.3"/>
+        <mu2 value="0.3"/>
     </gazebo>
 </robot>
